File: TP4056/TP4056.kicad_sch (KiCad schematic)
At the start: 5 parts, among them J1 USB_B_Micro, U1 TP4056-42-ESOP8, U2 DW01A

Commit message: schematics completed
Parts:
- added C2: 0.1uf, symbol Device:C
- added D1: Green LED, symbol Device:LED
- added D2: Red LED, symbol Device:LED
- added J2: B +, symbol Connector:Conn_01x01_Pin
- added J3: B -, symbol Connector:Conn_01x01_Pin
- added J4: OUT -, symbol Connector:Conn_01x01_Pin
- added J5: OUT +, symbol Connector:Conn_01x01_Pin
- added Q1: FDS9926A, Package_SO:SOIC-8_3.9x4.9mm_P1.27mm, symbol Transistor_FET:FDS9926A
- added R2: 100 ohm, symbol Device:R
- added R3: 1K2, symbol Device:R
- added R4, R5: R, symbol Device:R
- C1: value C -> 10uf
Connections:
- net at U2.1 (OD): now also Q1.2 (G1)
- net at U2.2 (CS): now also R3.1
- net at U2.3 (OC): now also Q1.4 (G2)
- net VDD: now reaches U2.5 (VCC)
- net VDD: now also U1.5 (BAT), C2.1, J5.1 (Pin_1), R2.2
- net at U2.6 (GND): now also C2.2, J3.1 (Pin_1), Q1.1 (S1)
- net +5V: now reaches J1.1 (VBUS)
- net +5V: now also C1.1, U1.4 (V_{CC}), U1.8 (CE), D1.2 (A), D2.2 (A)
- net GND: now reaches J1.5 (GND)
- net GND: now also C1.2, J1.SH (Shield), R1.2, U1.1 (TEMP), U1.3 (GND), U1.9 (EPAD), J4.1 (Pin_1), Q1.3 (S2), R3.2
- net at R1.1: now also U1.2 (PROG)
- net STDBY: now reaches U1.6 (~{STDBY})
- net STDBY: now also R4.2
- net CHRG: now reaches U1.7 (~{CHRG})
- net CHRG: now also R5.2
- new net: Q1.5 (D2), Q1.6 (D2), Q1.7 (D1), Q1.8 (D1)
- new net: J2.1 (Pin_1), R2.1
- new net: D2.1 (K), R5.1
- new net: D1.1 (K), R4.1
- no-connect marks 0 -> 3
Other:
- note added: "USB Power Supply"
- moved on the sheet: C1, J1, R1, U1, U2

Commit message: updated
Parts:
- C1, C2: footprint (none) -> Capacitor_SMD:C_0805_2012Metric
- D1, D2: footprint (none) -> LED_THT:LED_D1.8mm_W3.3mm_H2.4mm
- J1: footprint (none) -> Connector_USB:USB_Micro-B_Amphenol_10118194-0001LF_Horizontal
- J2, J3: footprint (none) -> Connector_Wire:SolderWirePad_1x01_SMD_1x2mm
- J4, J5: footprint (none) -> Connector_Wire:SolderWirePad_1x01_SMD_3x6mm
- R1, R2, R3: footprint (none) -> Resistor_THT:R_Axial_DIN0204_L3.6mm_D1.6mm_P5.08mm_Horizontal
- R4, R5: value R -> 1K; footprint (none) -> Resistor_THT:R_Axial_DIN0204_L3.6mm_D1.6mm_P5.08mm_Horizontal
Changed lines of the file:
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@@
+	)
+	(junction
+		(at 59.69 111.76)
+		(diameter 0)
+		(color 0 0 0 0)
 	)
 	(junction
@@
 	(wire
 		(pts
-			(xy 62.23 111.76) (xy 49.53 111.76)
+			(xy 62.23 111.76) (xy 59.69 111.76)
 		)
 		(stroke
@@
 	(wire
 		(pts
+			(xy 59.69 111.76) (xy 49.53 111.76)
+		)
+		(stroke
+			(width 0)
+			(type default)
+		)
+	)
+	(wire
+		(pts
 			(xy 44.45 40.64) (xy 53.34 40.64)
 		)
@@
 	(wire
 		(pts
+			(xy 59.69 110.49) (xy 59.69 111.76)
+		)
+		(stroke
+			(width 0)
+			(type default)
+		)
+	)
+	(wire
+		(pts
 			(xy 137.16 53.34) (xy 137.16 54.61)
 		)
@@
 	(wire
 		(pts
-			(xy 93.98 115.57) (xy 93.98 100.33)
-		)
-		(stroke
-			(width 0)
-			(type default)
-		)
-	)
-	(wire
-		(pts
 			(xy 193.04 41.91) (xy 200.66 41.91)
 		)
@@
 		(pts
 			(xy 36.83 115.57) (xy 49.53 115.57)
+		)
+		(stroke
+			(width 0)
+			(type default)
+		)
+	)
+	(wire
+		(pts
+			(xy 93.98 100.33) (xy 93.98 115.57)
 		)
 		(stroke
@@
 			)
 		)
-		(property "Footprint" ""
+		(property "Footprint" "Connector_USB:USB_Micro-B_Amphenol_10118194-0001LF_Horizontal"
 			(at 40.64 46.99 0)
 			(hide yes)
@@
 			)
 		)
-		(property "Footprint" ""
+		(property "Footprint" "Resistor_THT:R_Axial_DIN0204_L3.6mm_D1.6mm_P5.08mm_Horizontal"
 			(at 131.572 46.99 90)
 			(hide yes)
@@
 			)
 		)
-		(property "Footprint" ""
+		(property "Footprint" "Connector_Wire:SolderWirePad_1x01_SMD_1x2mm"
 			(at 31.75 115.57 0)
 			(hide yes)
@@
 			)
 		)
-		(property "Footprint" ""
+		(property "Footprint" "Capacitor_SMD:C_0805_2012Metric"
 			(at 50.4952 107.95 0)
 			(hide yes)
@@
 			)
 		)
-		(property "Footprint" ""
+		(property "Footprint" "Connector_Wire:SolderWirePad_1x01_SMD_1x2mm"
 			(at 31.75 95.25 0)
 			(hide yes)
@@
 				(path "/2fa4873c-1948-4884-98fa-e1999aa5379e"
 					(reference "J2")
+					(unit 1)
+				)
+			)
+		)
+	)
+	(symbol
+		(lib_id "power:PWR_FLAG")
+		(at 59.69 110.49 0)
+		(unit 1)
+		(body_style 1)
+		(exclude_from_sim no)
+		(in_bom yes)
+		(on_board yes)
+		(in_pos_files yes)
+		(dnp no)
+		(property "Reference" "#FLG01"
+			(at 59.69 108.585 0)
+			(hide yes)
+			(show_name no)
+			(do_not_autoplace no)
+			(effects
+				(font
+					(size 1.27 1.27)
+				)
+			)
+		)
+		(property "Value" "PWR_FLAG"
+			(at 59.436 102.108 90)
+			(show_name no)
+			(do_not_autoplace no)
+			(effects
+				(font
+					(size 1.27 1.27)
+				)
+			)
+		)
+		(property "Footprint" ""
+			(at 59.69 110.49 0)
+			(hide yes)
+			(show_name no)
+			(do_not_autoplace no)
+			(effects
+				(font
+					(size 1.27 1.27)
+				)
+			)
+		)
+		(property "Datasheet" ""
+			(at 59.69 110.49 0)
+			(hide yes)
+			(show_name no)
+			(do_not_autoplace no)
+			(effects
+				(font
+					(size 1.27 1.27)
+				)
+			)
+		)
+		(property "Description" "Special symbol for telling ERC where power comes from"
+			(at 59.69 110.49 0)
+			(hide yes)
+			(show_name no)
+			(do_not_autoplace no)
+			(effects
+				(font
+					(size 1.27 1.27)
+				)
+			)
+		)
+		(pin "1"
+		)
+		(instances
+			(project "TP4056"
+				(path "/2fa4873c-1948-4884-98fa-e1999aa5379e"
+					(reference "#FLG01")
 					(unit 1)
 				)
@@
 			)
 		)
-		(property "Footprint" ""
+		(property "Footprint" "LED_THT:LED_D1.8mm_W3.3mm_H2.4mm"
 			(at 233.68 41.91 0)
 			(hide yes)
@@
 			)
 		)
-		(property "Footprint" ""
+		(property "Footprint" "LED_THT:LED_D1.8mm_W3.3mm_H2.4mm"
 			(at 215.9 41.91 0)
 			(hide yes)
@@
 			)
 		)
-		(property "Footprint" ""
+		(property "Footprint" "Resistor_THT:R_Axial_DIN0204_L3.6mm_D1.6mm_P5.08mm_Horizontal"
 			(at 87.63 102.108 90)
 			(hide yes)
@@
 			)
 		)
-		(property "Footprint" ""
+		(property "Footprint" "Connector_Wire:SolderWirePad_1x01_SMD_3x6mm"
 			(at 55.88 85.09 0)
 			(hide yes)
@@
 			)
 		)
-		(property "Footprint" ""
+		(property "Footprint" "Resistor_THT:R_Axial_DIN0204_L3.6mm_D1.6mm_P5.08mm_Horizontal"
 			(at 43.18 97.028 90)
 			(hide yes)
@@
 			)
 		)
-		(property "Value" "R"
+		(property "Value" "1K"
 			(at 203.454 47.498 90)
 			(show_name no)
@@
 			)
 		)
-		(property "Footprint" ""
+		(property "Footprint" "Resistor_THT:R_Axial_DIN0204_L3.6mm_D1.6mm_P5.08mm_Horizontal"
 			(at 204.47 40.132 90)
 			(hide yes)
@@
 			)
 		)
-		(property "Footprint" ""
+		(property "Footprint" "Capacitor_SMD:C_0805_2012Metric"
 			(at 54.3052 48.26 0)
 			(hide yes)
@@
 			)
 		)
-		(property "Value" "R"
+		(property "Value" "1K"
 			(at 245.872 47.244 90)
 			(show_name no)
@@
 			)
 		)
-		(property "Footprint" ""
+		(property "Footprint" "Resistor_THT:R_Axial_DIN0204_L3.6mm_D1.6mm_P5.08mm_Horizontal"
 			(at 245.11 43.688 90)
 			(hide yes)
@@
 			)
 		)
-		(property "Footprint" ""
+		(property "Footprint" "Connector_Wire:SolderWirePad_1x01_SMD_3x6mm"
 			(at 93.98 85.09 0)
 			(hide yes)
