File: TP4056/TP4056.kicad_pcb (KiCad board)
At the start: 2 copper layers, 17 parts, among them J1 USB_B_Micro, J2 B +, J3 B -, J4 OUT -, J5 OUT +, Q1 FDS9926A, U1 TP4056-42-ESOP8, U2 DW01A

Commit message: pcb design adjustments
Parts:
- moved J4 82.9 mm to (163.0, 106.5)
- moved J3 82.1 mm to (163.0, 111.0)
- moved Q1 80.0 mm to (150.1, 109.5), turned to 90 degrees
- moved R1 78.7 mm to (135.0, 114.0), turned to -90 degrees
- moved J2 75.4 mm to (162.9, 113.6)
- moved J5 75.4 mm to (162.9, 118.1), turned to -90 degrees
- moved R2 74.5 mm to (153.5, 116.0)
- moved J1 71.6 mm to (125.3, 108.0)
- moved U1 70.0 mm to (136.9, 109.0), turned to 90 degrees
- moved C1 68.8 mm to (132.0, 107.5)
- moved R3 68.8 mm to (145.5, 103.5), turned to 0 degrees
- moved U2 67.8 mm to (143.6, 108.0), turned to 180 degrees
- moved C2 66.4 mm to (142.5, 112.0)
- moved R4 60.9 mm to (132.4, 102.5)
- moved D1 52.8 mm to (129.5, 99.0), turned to 180 degrees
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Routing:
- net /VDD: track 0.00 -> 39.4 mm
- net +5V: track 0.00 -> 38.0 mm
- net Net-(J3-Pin_1): track 0.72 -> 28.7 mm
- net Net-(D2-K): track 0.00 -> 14.3 mm
- net Net-(J2-Pin_1): track 0.00 -> 10.4 mm
- net /CHRG: track 0.00 -> 9.25 mm
- net Net-(Q1B-G2): track 0.57 -> 9.51 mm
- net Net-(U2-CS): track 0.00 -> 5.76 mm
- net Net-(Q1A-G1): track 0.79 -> 6.35 mm
- net Net-(D1-K): track 0.00 -> 4.73 mm
- net /STDBY: track 0.00 -> 4.02 mm
- net Net-(U1-PROG): track 0.00 -> 3.02 mm

Commit message: pcb design update
Routing:
- net Net-(Q1A-D1-Pad7): track 0.00 -> 3.81 mm
- added copper zone on F.Cu, net GND
Other:
- board outline added: 47 x 30 mm
Changed lines of the file:
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@@
 			(net "GND")
 			(pintype "passive")
+			(zone_connect 2)
 		)
 		(embedded_fonts no)
@@
 		)
 		(property "Value" "OUT +"
-			(at 0 2.54 90)
+			(at 0 -4.57 90)
 			(layer "F.Fab")
 			(effects
@@
 			(pinfunction "TEMP_1")
 			(pintype "input")
+			(zone_connect 2)
 		)
 		(pad "2" smd roundrect
@@
 			(pinfunction "GND_3")
 			(pintype "power_in")
+			(zone_connect 2)
 		)
 		(pad "4" smd roundrect
@@
 			(at -0.7 -1.2 90)
 			(size 0.5 0.5)
-			(drill 0.2)
+			(drill 0.3)
 			(property pad_prop_heatsink)
 			(layers "*.Cu")
@@
 			(at -0.7 0 90)
 			(size 0.5 0.5)
-			(drill 0.2)
+			(drill 0.3)
 			(property pad_prop_heatsink)
 			(layers "*.Cu")
@@
 			(at -0.7 1.2 90)
 			(size 0.5 0.5)
-			(drill 0.2)
+			(drill 0.3)
 			(property pad_prop_heatsink)
 			(layers "*.Cu")
@@
 			(at 0.7 -1.2 90)
 			(size 0.5 0.5)
-			(drill 0.2)
+			(drill 0.3)
 			(property pad_prop_heatsink)
 			(layers "*.Cu")
@@
 			(at 0.7 0 90)
 			(size 0.5 0.5)
-			(drill 0.2)
+			(drill 0.3)
 			(property pad_prop_heatsink)
 			(layers "*.Cu")
@@
 			(at 0.7 1.2 90)
 			(size 0.5 0.5)
-			(drill 0.2)
+			(drill 0.3)
 			(property pad_prop_heatsink)
 			(layers "*.Cu")
@@
 		)
 		(property "Value" "OUT -"
-			(at 0 2.54 90)
+			(at 0 4 90)
 			(layer "F.Fab")
 			(effects
@@
 			(net "GND")
 			(pintype "passive")
+			(zone_connect 2)
 		)
 		(embedded_fonts no)
@@
 		(tags "LED")
 		(property "Reference" "D1"
-			(at 1.77 -2.26 0)
+			(at 1 -2.5 0)
 			(layer "F.SilkS")
 			(effects
@@
 			(pinfunction "K_1")
 			(pintype "passive")
+			(zone_connect 0)
 		)
 		(pad "2" thru_hole circle
@@
 			(pinfunction "A_2")
 			(pintype "passive")
+			(zone_connect 0)
 		)
 		(embedded_fonts no)
@@
 			(pinfunction "GND_5")
 			(pintype "power_out")
+			(zone_connect 2)
 		)
 		(pad "SH" thru_hole oval
@@
 			(pinfunction "Shield_SH")
 			(pintype "passive")
+			(zone_connect 2)
 		)
 		(pad "SH" smd roundrect
@@
 			(pinfunction "Shield_SH")
 			(pintype "passive")
+			(zone_connect 2)
 		)
 		(pad "SH" smd roundrect
@@
 			(pinfunction "Shield_SH")
 			(pintype "passive")
+			(zone_connect 2)
 		)
 		(pad "SH" smd roundrect
@@
 		)
 	)
+	(gr_rect
+		(start 122.5 91)
+		(end 169.5 121)
+		(stroke
+			(width 0.05)
+			(type default)
+		)
+		(fill no)
+		(layer "Edge.Cuts")
+	)
 	(segment
 		(start 148.19 111.95)
@@
 	)
 	(segment
+		(start 150.73 107)
+		(end 152 107)
+		(width 0.2)
+		(layer "F.Cu")
+		(net "Net-(Q1A-D1-Pad7)")
+	)
+	(segment
+		(start 148.19 107)
+		(end 149.46 107)
+		(width 0.2)
+		(layer "F.Cu")
+		(net "Net-(Q1A-D1-Pad7)")
+	)
+	(segment
+		(start 149.46 107)
+		(end 150.73 107)
+		(width 0.2)
+		(layer "F.Cu")
+		(net "Net-(Q1A-D1-Pad7)")
+	)
+	(segment
 		(start 127.5 93.5)
 		(end 128 93)
@@
 		(net "/CHRG")
 	)
+	(zone
+		(net "GND")
+		(layer "F.Cu")
+		(hatch edge 0.5)
+		(connect_pads yes
+			(clearance 0.5)
+		)
+		(min_thickness 0.25)
+		(fill yes
+			(thermal_gap 0.5)
+			(thermal_bridge_width 0.5)
+			(island_removal_mode 0)
+		)
+		(polygon
+			(pts
+				(xy 122.5 91) (xy 122.5 121) (xy 169.546105 121) (xy 169.546105 91)
+			)
+		)
+	)
 	(embedded_fonts no)

Commit message: connections completed
Routing:
- net GND: track 0.00 -> 5.65 mm, vias 0 -> 6
Changed lines of the file:
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@@
 		)
 		(property "Value" "Red LED"
-			(at -4.73 0 0)
+			(at 10 -2 0)
 			(layer "F.Fab")
 			(effects
@@
 		)
 		(property "Value" "OUT +"
-			(at 0 -4.57 90)
+			(at -0.61 -4.57 90)
 			(layer "F.Fab")
 			(effects
@@
 		)
 		(property "Value" "OUT -"
-			(at 0 4 90)
+			(at 1 4.5 90)
 			(layer "F.Fab")
 			(effects
@@
 		)
 		(property "Value" "USB_B_Micro"
-			(at 0 5.2 90)
+			(at 6 -3.7 90)
 			(layer "F.Fab")
 			(effects
@@
 		(net "Net-(Q1A-G1)")
 	)
+	(via
+		(at 129 108)
+		(size 0.6)
+		(drill 0.3)
+		(layers "F.Cu" "B.Cu")
+		(free yes)
+		(net "GND")
+	)
+	(via
+		(at 150.5 114.5)
+		(size 0.6)
+		(drill 0.3)
+		(layers "F.Cu" "B.Cu")
+		(free yes)
+		(net "GND")
+	)
+	(via
+		(at 129 105)
+		(size 0.6)
+		(drill 0.3)
+		(layers "F.Cu" "B.Cu")
+		(free yes)
+		(net "GND")
+	)
+	(via
+		(at 150.73 111.95)
+		(size 0.6)
+		(drill 0.3)
+		(layers "F.Cu" "B.Cu")
+		(net "GND")
+	)
+	(via
+		(at 150.5 114.5)
+		(size 0.6)
+		(drill 0.3)
+		(layers "F.Cu" "B.Cu")
+		(free yes)
+		(net "GND")
+	)
+	(via
+		(at 129 108)
+		(size 0.6)
+		(drill 0.3)
+		(layers "F.Cu" "B.Cu")
+		(free yes)
+		(net "GND")
+	)
+	(segment
+		(start 150.73 114.27)
+		(end 150.73 111.95)
+		(width 0.2)
+		(layer "B.Cu")
+		(net "GND")
+	)
+	(segment
+		(start 150.5 114.5)
+		(end 150.73 114.27)
+		(width 0.2)
+		(layer "B.Cu")
+		(net "GND")
+	)
+	(segment
+		(start 129 105)
+		(end 129 108)
+		(width 0.2)
+		(layer "B.Cu")
+		(net "GND")
+	)
 	(segment

Commit message: gerber_files
Routing:
- net GND: track 5.65 -> 5.16 mm, vias 6 -> 4
Other:
- board size 47 x 30 mm -> 44.5 x 30 mm
Changed lines of the file:
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@@
 		(tags "MeasurementPoint Square SMDPad 3mmx6mm ")
 		(property "Reference" "J5"
-			(at 0.055 -5.475 90)
+			(at -1.11 4.43 90)
 			(layer "F.SilkS")
 			(effects
@@
 		)
 		(property "Value" "OUT +"
-			(at -0.61 -4.57 90)
+			(at 1.39 5.43 180)
 			(layer "F.Fab")
 			(effects
@@
 		)
 		(property "Value" "OUT -"
-			(at 1 4.5 90)
+			(at 6 -0.5 90)
 			(layer "F.Fab")
 			(effects
@@
 	(gr_rect
 		(start 122.5 91)
-		(end 169.5 121)
+		(end 167 121)
 		(stroke
 			(width 0.05)
@@
 	)
 	(via
-		(at 150.5 114.5)
-		(size 0.6)
-		(drill 0.3)
-		(layers "F.Cu" "B.Cu")
-		(free yes)
-		(net "GND")
-	)
-	(via
-		(at 129 105)
+		(at 151 114.5)
 		(size 0.6)
 		(drill 0.3)
@@
 	)
 	(via
-		(at 150.5 114.5)
+		(at 129 105.5)
 		(size 0.6)
 		(drill 0.3)
@@
 		(net "GND")
 	)
-	(via
-		(at 129 108)
-		(size 0.6)
-		(drill 0.3)
-		(layers "F.Cu" "B.Cu")
-		(free yes)
-		(net "GND")
-	)
-	(segment
-		(start 150.73 114.27)
-		(end 150.73 111.95)
+	(segment
+		(start 150.73 111.95)
+		(end 150.73 114.23)
 		(width 0.2)
 		(layer "B.Cu")
@@
 	)
 	(segment
-		(start 150.5 114.5)
-		(end 150.73 114.27)
+		(start 150.73 114.23)
+		(end 151 114.5)
 		(width 0.2)
 		(layer "B.Cu")
@@
 	)
 	(segment
-		(start 129 105)
+		(start 129 105.5)
 		(end 129 108)
 		(width 0.2)
@@
 		(polygon
 			(pts
-				(xy 122.5 91) (xy 122.5 121) (xy 169.546105 121) (xy 169.546105 91)
-			)
-		)
+				(xy 122.5 91) (xy 122.5 121) (xy 167 121) (xy 167 91)
+			)
+		)
